Commit message: Rename top_mount to mid_mount to stay consistent with the Boxer 2.4 URDF

File: boxer_franka_description/urdf/boxer_panda_description.urdf.xacro (robot description, xacro)
@@ -2,5 +2,5 @@
 <robot xmlns:xacro="http://ros.org/wiki/xacro">
   <joint name="arm_mount_joint" type="fixed">
-    <parent link="top_mount" />
+    <parent link="mid_mount" />
     <child link="arm_mount_link" />
     <origin xyz="$(optenv BOXER_FRANKA_XYZ 0.21 0.0 0.0)" rpy="$(optenv BOXER_FRANKA_RPY 0 0 0)"/>

File: boxer_franka_description/urdf/boxer_panda_hand_description.urdf.xacro (robot description, xacro)
@@ -2,5 +2,5 @@
 <robot xmlns:xacro="http://ros.org/wiki/xacro">
   <joint name="arm_mount_joint" type="fixed">
-    <parent link="top_mount" />
+    <parent link="mid_mount" />
     <child link="arm_mount_link" />
     <origin xyz="$(optenv BOXER_KINOVA_XYZ 0.21 0.0 0.0)" rpy="$(optenv BOXER_KINOVA_RPY 0 0 0)"/>

File: boxer_kinova_description/urdf/boxer_gen3_description.urdf.xacro (robot description, xacro)
@@ -10,5 +10,5 @@
   <xacro:load_robot arm="$(arg arm)" gripper="$(arg gripper)" dof="$(arg dof)" vision="$(arg vision)" sim="$(arg sim)" prefix="$(arg prefix)" />
   <joint name="arm_mount_joint" type="fixed">
-    <parent link="top_mount" />
+    <parent link="mid_mount" />
     <child link="kinova_arm_base_link" />
     <origin xyz="$(optenv BOXER_KINOVA_XYZ 0.21 0.0 0.0)" rpy="$(optenv BOXER_KINOVA_RPY 0 0 0)"/>

File: boxer_kinova_description/urdf/boxer_gen3_robotiq_2f_140_description.urdf.xacro (robot description, xacro)
@@ -10,5 +10,5 @@
   <xacro:load_robot arm="$(arg arm)" gripper="$(arg gripper)" dof="$(arg dof)" vision="$(arg vision)" sim="$(arg sim)" prefix="$(arg prefix)" />
   <joint name="arm_mount_joint" type="fixed">
-    <parent link="top_mount" />
+    <parent link="mid_mount" />
     <child link="kinova_arm_base_link" />
     <origin xyz="$(optenv BOXER_KINOVA_XYZ 0.21 0.0 0.0)" rpy="$(optenv BOXER_KINOVA_RPY 0 0 0)"/>

File: boxer_kinova_description/urdf/boxer_gen3_robotiq_2f_85_description.urdf.xacro (robot description, xacro)
@@ -10,5 +10,5 @@
   <xacro:load_robot arm="$(arg arm)" gripper="$(arg gripper)" dof="$(arg dof)" vision="$(arg vision)" sim="$(arg sim)" prefix="$(arg prefix)" />
   <joint name="arm_mount_joint" type="fixed">
-    <parent link="top_mount" />
+    <parent link="mid_mount" />
     <child link="kinova_arm_base_link" />
     <origin xyz="$(optenv BOXER_KINOVA_XYZ 0.21 0.0 0.0)" rpy="$(optenv BOXER_KINOVA_RPY 0 0 0)"/>

File: boxer_kinova_description/urdf/boxer_kinova_description.urdf.xacro (robot description, xacro)
@@ -2,5 +2,5 @@
 <robot xmlns:xacro="http://ros.org/wiki/xacro">
   <joint name="arm_mount_joint" type="fixed">
-    <parent link="top_mount" />
+    <parent link="mid_mount" />
     <child link="arm_mount_link" />
     <origin xyz="$(optenv BOXER_KINOVA_XYZ 0.21 0.0 0.0)" rpy="$(optenv BOXER_KINOVA_RPY 0 0 0)"/>

File: boxer_manipulation_description/urdf/boxer_upper_mount.urdf.xacro (robot description, xacro)
@@ -19,5 +19,5 @@
     <joint name="${name}_support_joint" type="fixed">
       <xacro:insert_block name="position"/>
-      <parent link="top_mount" />
+      <parent link="mid_mount" />
       <child link="${name}_support_link" />
     </joint>
@@ -41,5 +41,5 @@
     <joint name="${name}_upper_joint" type="fixed">
       <xacro:insert_block name="position"/>
-      <parent link="top_mount" />
+      <parent link="mid_mount" />
       <child link="${name}_upper_mount" />
     </joint>
@@ -63,5 +63,5 @@
     <joint name="${name}_upper_joint" type="fixed">
       <xacro:insert_block name="position"/>
-      <parent link="top_mount" />
+      <parent link="mid_mount" />
       <child link="${name}_upper_mount" />
     </joint>

File: boxer_ur_description/urdf/boxer_ur5_description.urdf.xacro (robot description, xacro)
@@ -2,5 +2,5 @@
 <robot xmlns:xacro="http://ros.org/wiki/xacro">
   <joint name="arm_mount_joint" type="fixed">
-    <parent link="top_mount" />
+    <parent link="mid_mount" />
     <child link="ur_arm_base_link" />
     <origin xyz="$(optenv BOXER_UR_XYZ 0.24 0.0 0.0)" rpy="$(optenv BOXER_UR_RPY 0 0 0)"/>

File: boxer_ur_description/urdf/boxer_ur5_e_description.urdf.xacro (robot description, xacro)
@@ -2,5 +2,5 @@
 <robot xmlns:xacro="http://ros.org/wiki/xacro">
   <joint name="arm_mount_joint" type="fixed">
-    <parent link="top_mount" />
+    <parent link="mid_mount" />
     <child link="ur_arm_base_link" />
     <origin xyz="$(optenv BOXER_UR_XYZ 0.24 0.0 0.0)" rpy="$(optenv BOXER_UR_RPY 0 0 0)"/>
