Commit message: Fix the tower material, fix a typo in the controller names

File: boxer_manipulation_description/urdf/boxer_dual_arm_tower.urdf.xacro (robot description, xacro)
@@ -4,5 +4,7 @@
     <link name="${prefix}_base_link">
       <visual>
-        <material name="black" />
+        <material name="black">
+          <color rgba="0 0 0 1" />
+        </material>
         <geometry>
           <mesh filename="package://boxer_manipulation_description/meshes/dual_arm_tower.stl" scale="0.001 0.001 0.001" />
